File: messing_around/part_explore/1_part_explore_proj/1_part_explore_proj.kicad_sch (KiCad schematic)
At the start: 2 parts, among them P1 USB_C_Plug_USB2.0, U1 ESP32-C3-WROOM-02

Commit message: messing around with the settings
Parts:
- added J1, J2: Conn_01x05, Connector_PinHeader_1.00mm:PinHeader_1x05_P1.00mm_Vertical, symbol Connector_Generic:Conn_01x05
- P1: footprint Connector_USB:USB_C_Plug_JAE_DX07P024AJ1 -> Connector_USB:USB_C_Receptacle_HRO_TYPE-C-31-M-12
Connections:
- net at U1.13 (IO18): no longer P1.A7 (D-)
- net at U1.14 (IO19): no longer P1.A6 (D+)
- net IO_3: now reaches U1.15 (IO3)
- net IO_3: now also J1.2 (Pin_2)
- net IO_2: now reaches U1.16 (IO2)
- net IO_2: now also J1.3 (Pin_3)
- net IO_1: now reaches U1.17 (IO1)
- net IO_1: now also J1.4 (Pin_4)
- net IO_0: now reaches U1.18 (IO0)
- net IO_0: now also J1.5 (Pin_5)
- net IO_4: now reaches U1.3 (IO4)
- net IO_4: now also J1.1 (Pin_1)
- net IO_5: now reaches U1.4 (IO5)
- net IO_5: now also J2.5 (Pin_5)
- net IO_6: now reaches U1.5 (IO6)
- net IO_6: now also J2.4 (Pin_4)
- net IO_7: now reaches U1.6 (IO7)
- net IO_7: now also J2.3 (Pin_3)
- net IO_8: now reaches U1.7 (IO8)
- net IO_8: now also J2.2 (Pin_2)
- net IO_9: now reaches U1.8 (IO9)
- net IO_9: now also J2.1 (Pin_1)
- new net USB_D+: P1.A6 (D+)
- new net USB_D-: P1.A7 (D-)
Other:
- moved on the sheet: P1, U1
