File: Learning/STM32_withBLT/STM32_withBLT/STM32_withBLT.kicad_sch (KiCad schematic)
At the start: 54 parts, among them J1 Conn_01x04, J2 Conn_Coaxial, J3 USB_C_Receptacle_USB2.0_16P, J4 Conn_01x10, SW1 SW_Push, U1 MIC5365-3.3YD5, U2 USBLC6-2SC6, U3 STM32WB55CEU6, X1 32kHz768, X2 32MHz

Commit message: initial stm32 bt pcb layout
Parts:
- removed R10, R6, R9: 100R, Capacitor_SMD:C_0402_1005Metric, symbol Device:R
- J1: footprint Connector_PinHeader_2.54mm:PinHeader_1x04_P2.54mm_Horizontal -> Connector_PinHeader_2.54mm:PinHeader_1x04_P2.54mm_Vertical
- J4: footprint Connector_PinHeader_2.54mm:PinHeader_1x10_P2.54mm_Horizontal -> Connector_PinHeader_2.54mm:PinHeader_1x10_P2.54mm_Vertical
- SW1: footprint Button_Switch_SMD:SW_SPST_Omron_B3FS-101xP -> Button_Switch_SMD:SW_SPST_FSMSM
Connections:
- net +3.3V: now also J1.4 (Pin_4), J4.2 (Pin_2), J4.3 (Pin_3); no longer J1.1 (Pin_1)
- net GND: now also J1.1 (Pin_1), J4.1 (Pin_1); no longer J1.4 (Pin_4)
- net GPIO1: no longer names the net of U3.28 (PB0)
- net GPIO2: no longer names the net of U3.29 (PB1)
- net GPIO3: no longer names the net of U3.19 (PB2)
Other:
- moved on the sheet: J1

Commit message: stm32 initial pcb layoout
Parts:
- added H1, H2, H3, H4: MountingHole, MountingHole:MountingHole_3.2mm_M3_Pad, symbol Mechanical:MountingHole
Connections:
- net BOOT_SW_OUT: now reaches R17.2, SW1.1
